File: pcb/mixer-fader/master/master.kicad_sch (KiCad schematic)
At the start: 0 parts

Commit message: Add master pcb
Parts:
- added J1: UART_SOCKET, Connector_JST:JST_XH_B4B-XH-A_1x04_P2.50mm_Vertical, symbol Connector:Conn_01x04_Socket
- added R1, R10, R11, R2, R3, R4, R5, R6, R7, R8, R9: 27, Resistor_SMD:R_0805_2012Metric, symbol Device:R
- added R12, R13: 100, Resistor_SMD:R_0805_2012Metric, symbol Device:R
- added U1: MixerFader_PogoPin_Male, PogoPinConnector:3x_PogoPinConnector_SMD_Male_01x05, symbol MixerFader_PogoPin:MixerFader_PogoPin_Male
Connections:
- new net: J1.2 (Pin_2), R12.2
- new net: J1.3 (Pin_3), R13.2
- new net +3V3: J1.1 (Pin_1), U1.1 (3.3V)
- new net GND: J1.4 (Pin_4), U1.2 (GND)
- new net Master_Display/DFF-CLK: R2.2, U1.5 (DISP_DFF_CLK)
- new net Master_Display/DFF-CLR: R3.2, U1.6 (DISP_DFF_CLR)
- new net Master_Display/DFF-D: R1.2
- new net Master_Display/DFF-Q: U1.4 (DISP_DFF_D)
- new net Master_Display/SPI-CLK: R5.2, U1.8 (DISP_SPI_CLK)
- new net Master_Display/SPI-DC: R6.2, U1.9 (DISP_DC)
- new net Master_Display/SPI-MOSI: R4.2, U1.7 (DISP_SPI_MOSI)
- new net Master_LevelMeter/CLK: R8.2, U1.11 (LED_CLK)
- new net Master_LevelMeter/DATA-IN: R7.2
- new net Master_LevelMeter/DATA-OUT: U1.10 (LED_DATA)
- new net Master_LevelMeter/LATCH: R9.2, U1.12 (LED_LATCH)
- new net Page_Encoder/CLK: R10.2, U1.14 (ENC_LATCH)
- new net Page_Encoder/DATA-IN: U1.13 (ENC_DATA)
- new net Page_Encoder/LATCH: R11.2, U1.15 (ENC_CLK)
- new net RP2040/GPIO0: R12.1
- new net RP2040/GPIO1: R13.1
- new net RP2040/GPIO15: U1.3 (DISP_LOOPBACK)
- new net RP2040/GPIO17: R1.1
- new net RP2040/GPIO18: R5.1
- new net RP2040/GPIO19: R4.1
- new net RP2040/GPIO2: R7.1
- new net RP2040/GPIO20: R6.1
- new net RP2040/GPIO21: R3.1
- new net RP2040/GPIO22: R2.1
- new net RP2040/GPIO3: R8.1
- new net RP2040/GPIO4: R9.1
- new net RP2040/GPIO6: R10.1
- new net RP2040/GPIO7: R11.1
Other:
- added sheet Master_Display (../common/sheets/display/display.kicad_sch)
- added sheet Master_LevelMeter (../common/sheets/level-meter/level-meter.kicad_sch)
- added sheet Page_Encoder (../common/sheets/encoder/encoder.kicad_sch)
- added sheet RP2040 (../common/sheets/rp2040/rp2040.kicad_sch)
- added sheet Volume_Encoder (../common/sheets/encoder/encoder.kicad_sch)
