File: pcb/mixer-fader/slave/slave.kicad_sch (KiCad schematic)
At the start: 0 parts

Commit message: Add slave pcb
Parts:
- added U1: MixerFader_PogoPin_Female, PogoPinConnector:3x_PogoPinConnector_SMD_Female_01x05_1_1, symbol MixerFader_PogoPin:MixerFader_PogoPin_Female
- added U2: MixerFader_PogoPin_Male, PogoPinConnector:3x_PogoPinConnector_SMD_Male_01x05, symbol MixerFader_PogoPin:MixerFader_PogoPin_Male
Connections:
- new net: U1.3 (DISP_LOOPBACK), U2.3 (DISP_LOOPBACK)
- new net +3V3: U1.1 (3.3V), U2.1 (3.3V)
- new net GND: U1.2 (GND), U2.2 (GND)
- new net Slave_Display/DFF-CLK: U1.5 (DISP_DFF_CLK), U2.5 (DISP_DFF_CLK)
- new net Slave_Display/DFF-CLR: U1.6 (DISP_DFF_CLR), U2.6 (DISP_DFF_CLR)
- new net Slave_Display/DFF-D: U1.4 (DISP_DFF_D)
- new net Slave_Display/DFF-Q: U2.4 (DISP_DFF_D)
- new net Slave_Display/SPI-CLK: U1.8 (DISP_SPI_CLK), U2.8 (DISP_SPI_CLK)
- new net Slave_Display/SPI-DC: U1.9 (DISP_DC), U2.9 (DISP_DC)
- new net Slave_Display/SPI-MOSI: U1.7 (DISP_SPI_MOSI), U2.7 (DISP_SPI_MOSI)
- new net Slave_Encoder/CLK: U1.15 (ENC_CLK), U2.15 (ENC_CLK)
- new net Slave_Encoder/DATA-IN: U2.13 (ENC_DATA)
- new net Slave_Encoder/DATA-OUT: U1.13 (ENC_DATA)
- new net Slave_Encoder/LATCH: U1.14 (ENC_LATCH), U2.14 (ENC_LATCH)
- new net Slave_LevelMeter/CLK: U1.11 (LED_CLK), U2.11 (LED_CLK)
- new net Slave_LevelMeter/DATA-IN: U1.10 (LED_DATA)
- new net Slave_LevelMeter/DATA-OUT: U2.10 (LED_DATA)
- new net Slave_LevelMeter/LATCH: U1.12 (LED_LATCH), U2.12 (LED_LATCH)
Other:
- added sheet Slave_Display (../common/sheets/display/display.kicad_sch)
- added sheet Slave_Encoder (../common/sheets/encoder/encoder.kicad_sch)
- added sheet Slave_LevelMeter (../common/sheets/level-meter/level-meter.kicad_sch)
