File: pcb/mixer-fader/common/sheets/display/display.kicad_sch (KiCad schematic)
At the start: 7 parts, among them U7 74LVC1G175, U8 ST7735_FPC

Commit message: Orderd PCB and Spacer, Window
Parts:
- renumbered C18 to C1, C19 to C2, C20 to C3, R22 to R1, R23 to R2, U7 to U3, U8 to U4
Changed lines of the file:
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@@
 		(dnp no)
 		(fields_autoplaced yes)
-		(property "Reference" "U7"
+		(property "Reference" "U3"
 			(at 59.69 19.05 0)
 			(effects
@@
 		(dnp no)
 		(fields_autoplaced yes)
-		(property "Reference" "U8"
+		(property "Reference" "U4"
 			(at 87.63 81.2799 0)
 			(effects
@@
 		(on_board yes)
 		(dnp no)
-		(property "Reference" "C20"
+		(property "Reference" "C3"
 			(at 66.04 101.6 90)
 			(effects
@@
 		(dnp no)
 		(fields_autoplaced yes)
-		(property "Reference" "C19"
+		(property "Reference" "C2"
 			(at 39.37 82.5499 0)
 			(effects
@@
 		(dnp no)
 		(fields_autoplaced yes)
-		(property "Reference" "R22"
+		(property "Reference" "R1"
 			(at 38.1 72.3899 0)
 			(effects
@@
 		(dnp no)
 		(fields_autoplaced yes)
-		(property "Reference" "R23"
+		(property "Reference" "R2"
 			(at 68.58 67.31 90)
 			(effects
@@
 		(on_board yes)
 		(dnp no)
-		(property "Reference" "C18"
+		(property "Reference" "C1"
 			(at 58.42 39.37 90)
 			(effects
