File: pcb/mixer-fader/common/sheets/encoder/encoder.kicad_sch (KiCad schematic)
At the start: 10 parts, among them U10 74LV165PW-Q100J, U9 EC11

Commit message: Orderd PCB and Spacer, Window
Parts:
- renumbered C21 to C5, C22 to C6, C23 to C7, R24 to R4, R25 to R5, R26 to R6, R27 to R7, R28 to R8, U9 to U7, U10 to U8
Changed lines of the file:
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@@
 		(dnp no)
 		(fields_autoplaced yes)
-		(property "Reference" "U10"
+		(property "Reference" "U8"
 			(at 160.8933 59.69 0)
 			(effects
@@
 		(on_board yes)
 		(dnp no)
-		(property "Reference" "C21"
+		(property "Reference" "C5"
 			(at 47.498 78.74 0)
 			(effects
@@
 		(dnp no)
 		(fields_autoplaced yes)
-		(property "Reference" "R28"
+		(property "Reference" "R8"
 			(at 58.42 58.4199 0)
 			(effects
@@
 		(dnp no)
 		(fields_autoplaced yes)
-		(property "Reference" "C22"
+		(property "Reference" "C6"
 			(at 59.69 78.7399 0)
 			(effects
@@
 		(dnp no)
 		(fields_autoplaced yes)
-		(property "Reference" "R26"
+		(property "Reference" "R6"
 			(at 96.52 29.2099 0)
 			(effects
@@
 		(dnp no)
 		(fields_autoplaced yes)
-		(property "Reference" "R25"
+		(property "Reference" "R5"
 			(at 58.42 29.2099 0)
 			(effects
@@
 		(dnp no)
 		(fields_autoplaced yes)
-		(property "Reference" "C23"
+		(property "Reference" "C7"
 			(at 180.34 88.8999 0)
 			(effects
@@
 		(dnp no)
 		(fields_autoplaced yes)
-		(property "Reference" "R27"
+		(property "Reference" "R7"
 			(at 46.99 58.4199 0)
 			(effects
@@
 		(dnp no)
 		(fields_autoplaced yes)
-		(property "Reference" "R24"
+		(property "Reference" "R4"
 			(at 46.99 29.2099 0)
 			(effects
@@
 		(dnp no)
 		(fields_autoplaced yes)
-		(property "Reference" "U9"
+		(property "Reference" "U7"
 			(at 78.105 30.48 0)
 			(effects
