File: pcb/mixer-fader/common/sheets/level-meter/level-meter.kicad_sch (KiCad schematic)
At the start: 4 parts, among them U13 TLC59283DBQR

Commit message: Orderd PCB and Spacer, Window
Parts:
- renumbered C27 to C4, R34 to R3, U13 to U5, U14 to U6
Changed lines of the file:
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@@
 		(dnp no)
 		(fields_autoplaced yes)
-		(property "Reference" "U13"
+		(property "Reference" "U5"
 			(at 60.96 30.48 0)
 			(effects
@@
 		(dnp no)
 		(fields_autoplaced yes)
-		(property "Reference" "U14"
+		(property "Reference" "U6"
 			(at 110.49 29.21 0)
 			(effects
@@
 		(on_board yes)
 		(dnp no)
-		(property "Reference" "R34"
+		(property "Reference" "R3"
 			(at 44.45 48.514 90)
 			(effects
@@
 		(dnp no)
 		(fields_autoplaced yes)
-		(property "Reference" "C27"
+		(property "Reference" "C4"
 			(at 24.13 49.5299 0)
 			(effects
